Commit message: first two weeks solution

File: src/hrwros_week2/urdf/hrwros_assignment1.xacro (robot description, xacro)
@@ -72,3 +72,9 @@
   </joint>
   <!-- Add your solution to assignment 1 here -->
+  <xacro:bin_urdf prefix="bin_2_"/>
+  <joint name="bin_2_joint" type="fixed">
+    <parent link="world_interface" />
+    <child link="bin_2_base_link" />
+    <origin xyz="2.5 1.8 0.0" rpy="0 0 0" />
+  </joint>
 </robot>

File: src/hrwros_week2/urdf/hrwros_assignment2.xacro (robot description, xacro)
@@ -72,3 +72,19 @@
   </joint>
   <!-- Add your solution to assignment 2 here -->
+  <link name="green_sphere">
+    <visual>
+      <origin xyz="0 0 0.5" />
+      <geometry>
+        <cylinder length="1" radius="0.4"/>
+      </geometry>
+      <material name="green_sphere_color">
+        <color rgba="${  0/255} ${155/255} ${ 70/255} 1.0" />
+      </material>
+    </visual>
+  </link>
+  <joint name="green_sphere_joint" type="fixed">
+    <origin xyz="5.8 -5.5 0.0" />
+    <parent link="world" />
+    <child link="green_sphere" />
+  </joint>
 </robot>

File: src/hrwros_week2/urdf/hrwros_assignment3.xacro (robot description, xacro)
@@ -65,10 +65,10 @@
   </joint>
   <!-- Update the below block for assignment 3 here -->
-  <xacro:include filename="$(find ur_description)/urdf/ur5.urdf.xacro"/>
-  <xacro:ur5_robot prefix="robot2_" joint_limited="true"/>
+  <xacro:include filename="$(find hrwros_week2)/urdf/robot/lrmate200ic_macro.xacro"/>
+  <xacro:fanuc_lrmate200ic prefix="robot2_"/>
   <joint name="robot2-robot2_pedestal_joint" type="fixed">
     <parent link="robot2_pedestal_link" />
     <child link="robot2_base_link" />
-    <origin xyz="0 0 0.6" rpy="0 0 ${radians(90)}" />
+    <origin xyz="0 0 0.6" rpy="0 0 ${radians(180)}" />
   </joint>
 </robot>
